Commit message: elizabeth_description: add footprint -> base_link to urdf

File: src/elizabeth_descriptions/urdf/elizabeth.xacro (robot description, xacro)
@@ -3,3 +3,9 @@
   <xacro:include filename="$(find abb_irb4600_support)/urdf/irb4600_40_255.xacro"/>
   <xacro:include filename="$(find elizabeth_descriptions)/urdf/t25_incl_all.xacro"/>
+  <link name="base_footprint"/>
+  <joint name="base_footprint_joint" type="fixed">
+    <parent link="base_footprint"/>
+    <child link="base_link"/>
+    <origin xyz="0 0 0.45" rpy="0 0 0"/>
+  </joint>
 </robot>
