Commit message: elizabeth_descriptions: fix references to meshes (package://)

File: src/elizabeth_descriptions/urdf/t25_incl_all.xacro (robot description, xacro)
@@ -5,5 +5,5 @@
     <visual>
       <geometry>
-        <mesh filename="file://$(find elizabeth_descriptions)/urdf/models/t25_incl_all.stl"/>
+        <mesh filename="package://elizabeth_descriptions/urdf/models/t25_incl_all.stl"/>
       </geometry>
       <origin xyz="0 0 0" rpy="0 0 0"/>
@@ -11,5 +11,5 @@
     <collision>
       <geometry>
-        <mesh filename="file://$(find elizabeth_descriptions)/urdf/models/t25_incl_all.stl"/>
+        <mesh filename="package://elizabeth_descriptions/urdf/models/t25_incl_all.stl"/>
       </geometry>
       <origin xyz="0 0 0" rpy="0 0 0"/>
