Commit message: fix(elizabeth_perception): dont run tf_static twice

File: src/elizabeth_perception/urdf/d405.urdf.xacro (robot description, xacro)
@@ -15,5 +15,6 @@
       use_nominal_extrinsics="$(arg use_nominal_extrinsics)"
       >
-    <origin xyz="0 0 0" rpy="0 0 0"/>
+    <!-- TODO: Needs calibration -->
+    <origin xyz="0.27275 0.025 0.058" rpy="0 0 0.2617994"/>
   </xacro:sensor_d405>
 </robot>
