Commit message: refactor: rename Elizabeth ROS packages

File: src/elizabeth_description/urdf/elizabeth.xacro (robot description, xacro)
@@ -4,5 +4,5 @@
   <xacro:arg name="rws_port" default="80"/>
   <xacro:include filename="$(find abb_irb4600_support)/urdf/irb4600_40_255.xacro"/>
-  <xacro:include filename="$(find elizabeth_descriptions)/urdf/t25_incl_all.xacro"/>
+  <xacro:include filename="$(find elizabeth_description)/urdf/t25_incl_all.xacro"/>
   <link name="base_footprint"/>
   <joint name="base_footprint_joint" type="fixed">

File: src/elizabeth_description/urdf/t25_incl_all.xacro (robot description, xacro)
@@ -5,5 +5,5 @@
     <visual>
       <geometry>
-        <mesh filename="package://elizabeth_descriptions/urdf/models/t25_incl_all.stl"/>
+        <mesh filename="package://elizabeth_description/urdf/models/t25_incl_all.stl"/>
       </geometry>
       <origin xyz="0 0 0" rpy="0 0 0"/>
@@ -11,5 +11,5 @@
     <collision>
       <geometry>
-        <mesh filename="package://elizabeth_descriptions/urdf/models/t25_incl_all.stl"/>
+        <mesh filename="package://elizabeth_description/urdf/models/t25_incl_all.stl"/>
       </geometry>
       <origin xyz="0 0 0" rpy="0 0 0"/>

File: src/elizabeth_moveit_config/config/elizabeth.urdf.xacro (robot description, xacro)
@@ -3,5 +3,5 @@
     <xacro:arg name="initial_positions_file" default="initial_positions.yaml" />
     <!-- Import elizabeth urdf file -->
-    <xacro:include filename="$(find elizabeth_descriptions)/urdf/elizabeth.xacro" />
+    <xacro:include filename="$(find elizabeth_description)/urdf/elizabeth.xacro" />
     <!-- Import control_xacro -->
     <xacro:include filename="elizabeth.ros2_control.xacro" />
